File: KiCAD_Project/instrumentation_amp.sch (KiCad schematic (older format))
At the start: 68 parts, among them J1 SPDT_SOLDER, J2 SPDT_SOLDER, J3 SPDT_SOLDER, J4 SPDT_SOLDER, J5 SP3T_SOLDER, J6 SP3T_SOLDER, P1 +VIN, P10 TXDR -OUT 2, P11 +15VDC, P12 +15VDC, P13 +15VDC, P14 -15VDC, P15 -15VDC, P16 -15VDC, P17 GND, P18 GND, P19 GND, P2 -VIN, P20 GND, P3 TXDR -IN 1, P4 TXDR -IN 1, P5 TXDR -IN 2, P6 TXDR -IN 2, P7 TXDR -OUT 1, P8 TXDR -OUT 1, P9 TXDR -OUT 2, U1 LM7815CT, U2 LM7915CT, U3 INA128, U4 INA128

Commit message: Change jumpers for better operation and rework the layout
Parts:
- removed P1: +VIN, symbol CONN_1
- removed P10, P9: TXDR -OUT 2, symbol CONN_1
- removed P11, P12, P13: +15VDC, symbol CONN_1
- removed P14, P15, P16: -15VDC, symbol CONN_1
- removed P17, P18, P19, P20: GND, symbol CONN_1
- removed P2: -VIN, symbol CONN_1
- removed P3, P4: TXDR -IN 1, symbol CONN_1
- removed P5, P6: TXDR -IN 2, symbol CONN_1
- removed P7, P8: TXDR -OUT 1, symbol CONN_1
- added P1, P2, P3, P4: CONN_5, symbol CONN_5
Connections:
- net labels added: A +IN, A +OUT, A -IN, A -OUT, B +IN, B +OUT, B -IN, B -OUT, VDD, VSS
- net labels removed: +15V, -15V
- wire segments 129 -> 148
Other:
- note removed: "Power Access Points\n\n"

Commit message: Add solder paste stencil files
Other:
- note added: "B"
- note removed: "A"
Changed lines of the file:
@@
 Sheet 1 1
 Title ""
-Date "12 nov 2014"
+Date "7 dec 2014"
 Rev ""
 Comp ""
@@
 Connection ~ 5700 4500
 Text Notes 9940 7890 0    60   ~ 0
-A
+B
 Text Notes 6650 7770 0    60   ~ 0
 Dual Channel Instrumentation Buffer/Amplifier - J.R. Leeman
